Commit message: working Ros2 controls plugin with query and command loop

File: ros2/urdf/rrbot/rrbot_lss_hardware_position_only.ros2_control.xacro (robot description, xacro)
@@ -4,10 +4,10 @@
     <ros2_control name="${name}" type="system">
       <hardware>
-        <plugin>lynxmotion/LynxmotionServoHardware</plugin>
+        <plugin>lynxmotion/LssBus</plugin>
         <param name="port">/dev/ttyUSB0</param>
-        <param name="baudrate">500000</param>
+        <param name="baudrate">921600</param>
         <param name="prefix">J</param>
       </hardware>
-      <joint name="J28">
+      <joint name="J0">
         <command_interface name="position">
           <param name="min">-1800</param>
@@ -18,5 +18,5 @@
         <state_interface name="current"/>
       </joint>
-      <joint name="J29">
+      <joint name="J5">
         <command_interface name="position">
           <param name="min">-1800</param>
